File: pcb/light-diffusion/light-diffusion.kicad_pcb (KiCad board)
At the start: 2 copper layers, 5 x 8 mm, 1 part

Commit message: pcbs and updated cad pushed up
Other:
- outline, holes or cut-outs redrawn
Changed lines of the file:
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@@
-(kicad_pcb (version 20211014) (generator pcbnew)
+(kicad_pcb (version 20221018) (generator pcbnew)
   (general
     (thickness 1.6)
@@
     (pcbplotparams
       (layerselection 0x00010fc_ffffffff)
+      (plot_on_all_layers_selection 0x0000000_00000000)
       (disableapertmacros false)
       (usegerberextensions false)
@@
       (usegerberadvancedattributes true)
       (creategerberjobfile true)
-      (svguseinch false)
+      (dashed_line_dash_ratio 12.000000)
+      (dashed_line_gap_ratio 3.000000)
       (svgprecision 6)
-      (excludeedgelayer true)
       (plotframeref false)
       (viasonmask false)
@@
       (drillshape 0)
       (scaleselection 1)
-      (outputdirectory "out/rev00/")
+      (outputdirectory "out/rev01/")
     )
   )
@@
     (attr board_only exclude_from_pos_files exclude_from_bom)
     (fp_text reference "G***" (at -6.8 0) (layer "F.SilkS") hide
-      (effects (font (size 1.524 1.524) (thickness 0.3)))
+        (effects (font (size 1.524 1.524) (thickness 0.3)))
     )
     (fp_text value "LOGO" (at 0.75 0) (layer "F.SilkS") hide
-      (effects (font (size 1.524 1.524) (thickness 0.3)))
+        (effects (font (size 1.524 1.524) (thickness 0.3)))
     )
-    (fp_poly (pts
+    (fp_poly
+      (pts
         (xy 5 5)
         (xy -5 5)
@@
         (xy -5 -5)
         (xy 5 -5)
-      ) (layer "F.Mask") (width 0) (fill solid))
-    (fp_poly (pts
+      )
+      (stroke (width 0) (type solid)) (fill solid) (layer "F.Mask"))
+    (fp_poly
+      (pts
         (xy 0.124383 -1.16212)
         (xy 0.138097 -1.160624)
@@
         (xy 0.106804 -1.162553)
         (xy 0.114079 -1.162752)
-      ) (layer "F.Mask") (width 0) (fill solid))
+      )
+      (stroke (width 0) (type solid)) (fill solid) (layer "F.Mask"))
   )
-  (gr_rect (start 0 -7) (end 5 -1) (layer "B.Mask") (width 0.1) (fill solid))
-  (gr_line (start 0 0) (end 5 0) (layer "Edge.Cuts") (width 0.1))
-  (gr_line (start 0 -8) (end 0 0) (layer "Edge.Cuts") (width 0.1))
-  (gr_line (start 3 -7.5) (end 5 -7.5) (layer "Edge.Cuts") (width 0.1))
-  (gr_line (start 5 0) (end 5 -7.5) (layer "Edge.Cuts") (width 0.1))
-  (gr_line (start 0 -8) (end 2.5 -8) (layer "Edge.Cuts") (width 0.1))
-  (gr_arc (start 3 -7.5) (mid 2.646447 -7.646447) (end 2.5 -8) (layer "Edge.Cuts") (width 0.1))
-  (zone (net 0) (net_name "") (layers F&B.Cu) (hatch edge 0.508)
+  (gr_rect (start 0 -7) (end 5 -1)
+    (stroke (width 0.1) (type solid)) (fill solid) (layer "B.Mask"))
+  (gr_line (start 0 0) (end 5 0)
+    (stroke (width 0.1) (type solid)) (layer "Edge.Cuts"))
+  (gr_line (start 0 -8) (end 0 0)
+    (stroke (width 0.1) (type solid)) (layer "Edge.Cuts"))
+  (gr_line (start 5 0) (end 5 -8)
+    (stroke (width 0.1) (type solid)) (layer "Edge.Cuts"))
+  (gr_line (start 0 -8) (end 5 -8)
+    (stroke (width 0.1) (type solid)) (layer "Edge.Cuts"))
+  (zone (net 0) (net_name "") (layers "F&B.Cu") (hatch edge 0.508)
     (connect_pads (clearance 0))
-    (min_thickness 0.254)
-    (keepout (tracks not_allowed) (vias not_allowed) (pads not_allowed ) (copperpour not_allowed) (footprints allowed))
+    (min_thickness 0.254) (filled_areas_thickness no)
+    (keepout (tracks not_allowed) (vias not_allowed) (pads not_allowed) (copperpour not_allowed) (footprints allowed))
     (fill (thermal_gap 0.508) (thermal_bridge_width 0.508))
     (polygon
