File: pcb/feeder-mobo-ott/feeder-mobo-ott.kicad_pcb (KiCad board)
At the start: 2 copper layers, 71.6 x 80 mm, 79 parts, among them J1 SWD_10, J2 PEEL_MOTOR, J3 DRIVE_MOTOR, J5 SPRING_FINGERS, J8 USART1, SW3 BACK_BTN, SW4 FWD_BTN, SW5 RESET_BTN, U1 AP63203WU, U2 MHS110FRGBCT, U3 STM32F030C8Tx, U4 AP63200WU, U6 MAX3078E, U7 DRV8837, U8 DRV8837, Y1 8MHz

Commit message: PVT 2u
Parts:
- added 1WIRE: TP_1WIRE, TestPoint:TestPoint_Pad_D2.0mm, F.Cu at (112.1, 114.2)
- added BOOT0: TP_BOOT0, TestPoint:TestPoint_Pad_D2.0mm, F.Cu at (60.5, 123.7)
- added G***: LOGO, mfg:logo_mask, B.Cu at (115.3, 58.8)
- added RS485+: TP_485+, TestPoint:TestPoint_Pad_D2.0mm, F.Cu at (107.8, 113.7)
- added RS485-: TP_485-, TestPoint:TestPoint_Pad_D2.0mm, F.Cu at (108.0, 107.7)
- added SW1: TP_SW1, TestPoint:TestPoint_Pad_D2.0mm, F.Cu at (89.2, 58.0)
- added SW2: TP_SW2, TestPoint:TestPoint_Pad_D2.0mm, F.Cu at (113.3, 58.5)
- R5: value 218k -> 215k
- moved G*** 2.22 mm to (69.8, 126.3)
Routing:
- net RS-485-: track 8.95 -> 26.5 mm, vias 0 -> 2
- net SW1: track 58.4 -> 65.9 mm
- net Net-(J5-Pin_5): track 3.99 -> 10.7 mm
- net RS-485+: track 14.5 -> 19.0 mm
- net BOOT0: track 45.3 -> 47.3 mm
- net SW2: track 62.9 -> 64.9 mm
- net +3V3: track 216.6 -> 215.9 mm
- net GND: vias 100 -> 206
Other:
- outline, holes or cut-outs redrawn
- board text added: "10v"
- board text added: "3v3"
- board text added: "D1"
- board text added: "D2"
- board text added: "ENC_A"
- board text added: "ENC_B"
- board text added: "Feeder OTT Mobo REV01 Opulo Inc."
- board text added: "GND"
- board text added: "P1"
- board text added: "P2"
- board text added: "RST"
- board text added: "SWCLK"
- board text added: "SWDIO"
- board text added: "VDC"
- board text removed: "LumenPnP 2u Feeder REV00b2 Opulo Inc."
