File: pcb/feeder-mobo-ott/feeder-mobo-ott.kicad_sch (KiCad schematic)
At the start: 77 parts, among them J1 SWD_10, J2 PEEL_MOTOR, J3 DRIVE_MOTOR, J5 SPRING_FINGERS, J8 USART1, SW3 BACK_BTN, SW4 FWD_BTN, SW5 RESET_BTN, U1 AP63203WU, U2 MHS110FRGBCT, U3 STM32F030C8Tx, U4 AP63200WU, U6 MAX3078E, U7 DRV8837, U8 DRV8837, Y1 8MHz

Commit message: PVT 2u
Parts:
- added TP15: TP_485-, TestPoint:TestPoint_Pad_D2.0mm, symbol Connector:TestPoint
- added TP16: TP_BOOT0, TestPoint:TestPoint_Pad_D2.0mm, symbol Connector:TestPoint
- added TP17: TP_SW1, TestPoint:TestPoint_Pad_D2.0mm, symbol Connector:TestPoint
- added TP18: TP_SW2, TestPoint:TestPoint_Pad_D2.0mm, symbol Connector:TestPoint
- added TP19: TP_1WIRE, TestPoint:TestPoint_Pad_D2.0mm, symbol Connector:TestPoint
- added TP2: TP_485+, TestPoint:TestPoint_Pad_D2.0mm, symbol Connector:TestPoint
- D3, D5, D6: LCSC (none) -> C2891607
- D7: LCSC (none) -> C41376091
- D9: LCSC (none) -> C24672
- J2: LCSC C2845379 -> C2845388
- J5: LCSC (none) -> C3035810
- L1: LCSC (none) -> C167751
- L3: LCSC (none) -> C6364790
- R14: LCSC (none) -> C17557
- R15, R16: LCSC (none) -> C114557
- R2, R3: LCSC (none) -> C107700
- R5: value 218k -> 215k
- SW3, SW4, SW5: LCSC (none) -> C115365
- U1: LCSC (none) -> C780769
- U2: LCSC (none) -> C496820
- U3: LCSC (none) -> C40053
- U4: LCSC (none) -> C2071868; LCSC # (none) -> C2071868
- U7, U8: LCSC (none) -> C39159
Connections:
- net BOOT0: now also TP16.1
- net RS-485+: now also TP2.1
- net RS-485-: now also TP15.1
- net SW1: now also TP17.1
- net SW2: now also TP18.1
- net at J5.5 (Pin_5), R14.2: now also TP19.1
Other:
- note removed: "120 Ohm termination resistor needed at the end of the bus"
- moved on the sheet: C6, D2, D9, J5, R14, R15, R16, R17, SW3, SW4, SW5, TP9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
